File: OtterPill.kicad_pcb (KiCad board)
At the start: 2 copper layers, 43.2 x 17.6 mm, 38 parts, among them J1 USB-c, J2 usb2, J3 1, J4 2, J5 SWD, SW1 SW_Push, U1 USBLC6-4, U2 STM32F072CBUx, U3 ACT4088, U4 FUSB302BMPX

Commit message: added gerber
Parts:
- removed the G*** at (42.4, 27.0)
- removed J2: usb2, Connector_USB:USB_Micro-B_Molex-105017-0001
- added G***: LOGO, otter:otter_laying_3411, B.Cu at (41.0, 26.9)
Routing:
- net USB_P: track 23.9 -> 20.7 mm, vias 4 -> 2
- net GND: track 31.1 -> 28.5 mm
- net USB_N: track 22.2 -> 19.9 mm
- net VBUS: vias 13 -> 12

Commit message: v1.2
Parts:
- moved R5 0.25 mm to (51.0, 33.1)
Routing:
- net GND: track 28.5 -> 22.3 mm, vias 52 -> 53

Commit message: updated PCB and gerber
Parts:
- removed G***: LOGO, otter:otter_laying_3411
- R1, R2: value 5k1 -> DNP
- R3, R4: value R -> 5k1
- R6: value TBD -> 16k
- R8, R9: value DNP -> 0
Connections:
- U1 pad 5: VBUS -> +3V3
Routing:
- net GND: track 22.3 -> 28.5 mm, vias 53 -> 48
- net +3V3: track 108.8 -> 114.9 mm, vias 7 -> 11
- net VBUS: track 35.9 -> 39.2 mm, vias 12 -> 10
- net 33: track 15.0 -> 14.1 mm
- net 31: track 23.4 -> 22.6 mm
- net INT_N: track 14.7 -> 14.8 mm, vias 4 -> 3
- net 32: track 20.0 -> 19.9 mm, vias 3 -> 2

Commit message: updated otterpill to V1.2
Parts:
- removed D3: SS310, Diode_SMD:D_SOD-123
- added C11: 10u 25V, Capacitor_SMD:C_0805_2012Metric, F.Cu at (54.7, 28.9)
- added J2: VBUS, Connector_PinHeader_2.54mm:PinHeader_1x01_P2.54mm_Vertical, F.Cu at (21.4, 21.8)
- added J6: GND, Connector_PinHeader_2.54mm:PinHeader_1x01_P2.54mm_Vertical, F.Cu at (21.4, 35.3)
- C1, C4: value 10u -> 10u 25V
- C10, C2, C3, C5, C6, C7, C8, C9: value 100n -> 100n 50V
- D1: value LED -> LED RED
- D2: value LED -> LED GREEN
- R10, R11, R3, R4, R5, R7: value 5k1 -> 3k3
- R12: value 5k1 -> 10k
- R6: value 16k -> 10k
- U2: value STM32F072CBUx -> STM32F072C8Tx; footprint Package_DFN_QFN:QFN-48-1EP_7x7mm_P0.5mm_EP5.6x5.6mm -> Package_QFP:LQFP-48_7x7mm_P0.5mm
- U3: value ACT4088 -> SY8201
- moved R12 16.0 mm to (52.8, 28.8), turned to 0 degrees
- moved C6 8.07 mm to (48.9, 31.0), turned to 180 degrees
- moved R7 4.59 mm to (49.5, 26.7), turned to 90 degrees
- moved C3 3.91 mm to (54.8, 23.3), turned to 0 degrees
- moved C9 3.80 mm to (49.3, 23.9)
- moved C1 3.18 mm to (51.9, 23.8), turned to 180 degrees
- moved R11 2.52 mm to (36.7, 25.8), turned to 90 degrees
- moved C2 2.34 mm to (51.2, 29.0)
- moved R6 1.91 mm to (52.8, 29.7), turned to 180 degrees
- moved U3 1.81 mm to (51.9, 26.5), turned to 0 degrees
- moved C5 1.43 mm to (49.4, 29.7), turned to 0 degrees
- moved L1 1.41 mm to (55.6, 25.6), turned to 270 degrees
- moved C4 1.28 mm to (56.5, 29.0)
- moved D4 1.19 mm to (47.3, 24.3), turned to 135 degrees
- moved C7 1.01 mm to (36.5, 27.7), turned to 270 degrees
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Connections:
- R12 pad 1: +3V3 -> VIN
- R12 pad 2: INT_N -> Net-(R12-Pad2)
- U3 pad 1: Net-(C3-Pad2) -> Net-(C3-Pad1)
- U3 pad 2: VIN -> GND
- U3 pad 3: Net-(U3-Pad3) -> Net-(R6-Pad2)
- U3 pad 4: Net-(R6-Pad2) -> Net-(R12-Pad2)
- U3 pad 5: GND -> VIN
- U3 pad 6: Net-(C3-Pad1) -> Net-(C3-Pad2)
Routing:
- net +3V3: track 114.9 -> 86.7 mm, vias 11 -> 4
- net GND: track 28.5 -> 10.6 mm, vias 48 -> 29
- net VBUS: track 39.2 -> 49.8 mm
- net Net-(C3-Pad1): track 1.75 -> 7.40 mm
- net Net-(R6-Pad2): track 2.52 -> 6.62 mm, vias 0 -> 2
- net 314: track 22.0 -> 26.0 mm
- net SWCLK: track 25.2 -> 22.0 mm
- net 49: track 5.89 -> 8.60 mm, vias 1 -> 0
- net SWDIO: track 25.2 -> 22.6 mm
- net Net-(R5-Pad1): track 19.4 -> 16.9 mm, vias 3 -> 2
- net 45: track 19.4 -> 17.1 mm, vias 2 -> 0
- net 44: track 18.1 -> 19.9 mm
- net 48: track 9.99 -> 8.30 mm, vias 1 -> 2
- net SDA: track 7.34 -> 5.67 mm
- net Net-(R12-Pad2): track 0.00 -> 1.45 mm
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
Commit message: updated otterpill to V1.2
Parts:
- L1: footprint Inductor_SMD:L_Taiyo-Yuden_MD-3030 -> Inductor_SMD:L_1210_3225Metric
- moved R6 2.66 mm to (50.2, 29.0), turned to 90 degrees
- moved C5 1.29 mm to (49.9, 30.9), turned to 270 degrees
- moved C3 1.17 mm to (53.7, 23.9), turned to 270 degrees
- moved C9 0.99 mm to (48.5, 23.2), turned to 135 degrees
- moved C6 0.76 mm to (48.9, 30.3), turned to 270 degrees
- moved L1 0.53 mm to (55.8, 25.1)
- moved R7 0.41 mm to (49.6, 27.1)
- moved C1 0.33 mm to (51.6, 23.9)
- moved D4 0.31 mm to (47.5, 24.5)
- moved U3 0.11 mm to (52.0, 26.5)
Routing:
- net +3V3: track 86.7 -> 97.3 mm
- net VBUS: track 49.8 -> 44.8 mm, vias 10 -> 9
- net Net-(R6-Pad2): track 6.62 -> 2.62 mm, vias 2 -> 0
- net Net-(C3-Pad1): track 7.40 -> 5.27 mm, vias 0 -> 2
- net VIN: track 23.8 -> 25.3 mm, vias 1 -> 2
- net Net-(C3-Pad2): track 0.00 -> 1.49 mm
- net INT_N: track 14.0 -> 14.9 mm
- net 47: track 11.5 -> 12.3 mm
- net 44: track 19.9 -> 19.3 mm
- net GND: vias 29 -> 40
Other:
- board text added: "PB6"
