File: OtterPill.sch (KiCad schematic (older format))
At the start: 37 parts, among them J1 USB-c, J2 usb2, J3 1, J4 2, J5 SWD, SW1 SW_Push, U1 USBLC6-4, U2 STM32F072CBUx, U3 ACT4088, U4 FUSB302BMPX

Commit message: added gerber
Parts:
- removed J2: usb2, Connector_USB:USB_Micro-B_Molex-105017-0001, symbol Connector:USB_B_Micro
Changed lines of the file:
@@
 EESchema Schematic File Version 4
-LIBS:stm32f072PrototypingBoard-cache
 EELAYER 29 0
 EELAYER END
@@
 $EndComp
 $Comp
-L Connector:USB_B_Micro J2
-U 1 1 5CC70E6B
-P 1350 4200
-F 0 "J2" H 1407 4667 50  0000 C CNN
-F 1 "usb2" H 1407 4576 50  0000 C CNN
-F 2 "Connector_USB:USB_Micro-B_Molex-105017-0001" H 1500 4150 50  0001 C CNN
-F 3 "~" H 1500 4150 50  0001 C CNN
-	1    1350 4200
-	1    0    0    -1
-$EndComp
-$Comp
-L power:VBUS #PWR0109
-U 1 1 5CC72249
-P 1650 4000
-F 0 "#PWR0109" H 1650 3850 50  0001 C CNN
-F 1 "VBUS" H 1665 4173 50  0000 C CNN
-F 2 "" H 1650 4000 50  0001 C CNN
-F 3 "" H 1650 4000 50  0001 C CNN
-	1    1650 4000
-	1    0    0    -1
-$EndComp
-$Comp
-L power:GND #PWR0110
-U 1 1 5CC7260A
-P 1350 4600
-F 0 "#PWR0110" H 1350 4350 50  0001 C CNN
-F 1 "GND" H 1355 4427 50  0000 C CNN
-F 2 "" H 1350 4600 50  0001 C CNN
-F 3 "" H 1350 4600 50  0001 C CNN
-	1    1350 4600
-	1    0    0    -1
-$EndComp
-$Comp
-L power:GND #PWR0111
-U 1 1 5CC728D9
-P 1250 4600
-F 0 "#PWR0111" H 1250 4350 50  0001 C CNN
-F 1 "GND" H 1255 4427 50  0000 C CNN
-F 2 "" H 1250 4600 50  0001 C CNN
-F 3 "" H 1250 4600 50  0001 C CNN
-	1    1250 4600
-	1    0    0    -1
-$EndComp
-Text GLabel 1650 4300 2    50   Input ~ 0
-USB_N
-Text GLabel 1650 4200 2    50   Input ~ 0
-USB_P
-$Comp
 L otter:USBLC6-4 U1

Commit message: v1.2
Parts:
- R6: value TBD -> 16k
Changed lines of the file:
@@
 EESchema Schematic File Version 4
+LIBS:OtterPill-cache
 EELAYER 29 0
 EELAYER END
@@
 P 8800 3200
 F 0 "R6" H 8859 3246 50  0000 L CNN
-F 1 "TBD" H 8859 3155 50  0000 L CNN
+F 1 "16k" H 8859 3155 50  0000 L CNN
 F 2 "Resistor_SMD:R_0402_1005Metric" H 8800 3200 50  0001 C CNN
 F 3 "~" H 8800 3200 50  0001 C CNN
@@
 F 3 "~" H 3150 3200 50  0001 C CNN
 	1    3150 3200
-	0    1    1    0
-$EndComp
-$Comp
-L Device:R_Small R11
-U 1 1 5CCA53F5
-P 3150 3300
-F 0 "R11" V 3254 3300 50  0000 C CNN
-F 1 "5k1" V 3345 3300 50  0000 C CNN
-F 2 "Resistor_SMD:R_0402_1005Metric" H 3150 3300 50  0001 C CNN
-F 3 "~" H 3150 3300 50  0001 C CNN
-	1    3150 3300
 	0    1    1    0
 $EndComp
@@
 Wire Wire Line
 	4750 3200 4750 2700
+$Comp
+L Device:R_Small R11
+U 1 1 5CCA53F5
+P 3150 3300
+F 0 "R11" V 3254 3300 50  0000 C CNN
+F 1 "5k1" V 3345 3300 50  0000 C CNN
+F 2 "Resistor_SMD:R_0402_1005Metric" H 3150 3300 50  0001 C CNN
+F 3 "~" H 3150 3300 50  0001 C CNN
+	1    3150 3300
+	0    1    1    0
+$EndComp
 $EndSCHEMATC

Commit message: updated PCB and gerber
Parts:
- R1, R2: value 5k1 -> DNP
- R3, R4: value R -> 5k1
- R8, R9: value DNP -> 0
Connections:
- net +3V3: now also U1.5 (VBUS)
- net VBUS: no longer U1.5 (VBUS)
Changed lines of the file:
@@
 EESchema Schematic File Version 4
 LIBS:OtterPill-cache
-EELAYER 29 0
+EELAYER 26 0
 EELAYER END
 $Descr A4 11693 8268
@@
 P 3300 2850
 F 0 "R1" V 3104 2850 50  0000 C CNN
-F 1 "5k1" V 3195 2850 50  0000 C CNN
+F 1 "DNP" V 3195 2850 50  0000 C CNN
 F 2 "Resistor_SMD:R_0402_1005Metric" H 3300 2850 50  0001 C CNN
 F 3 "~" H 3300 2850 50  0001 C CNN
@@
 P 3300 2950
 F 0 "R2" V 3404 2950 50  0000 C CNN
-F 1 "5k1" V 3495 2950 50  0000 C CNN
+F 1 "DNP" V 3495 2950 50  0000 C CNN
 F 2 "Resistor_SMD:R_0402_1005Metric" H 3300 2950 50  0001 C CNN
 F 3 "~" H 3300 2950 50  0001 C CNN
@@
 F 3 "" H 2700 4200 50  0001 C CNN
 	1    2700 4200
-	1    0    0    -1
-$EndComp
-$Comp
-L power:VBUS #PWR0113
-U 1 1 5CC748E3
-P 3300 4000
-F 0 "#PWR0113" H 3300 3850 50  0001 C CNN
-F 1 "VBUS" H 3315 4173 50  0000 C CNN
-F 2 "" H 3300 4000 50  0001 C CNN
-F 3 "" H 3300 4000 50  0001 C CNN
-	1    3300 4000
 	1    0    0    -1
 $EndComp
@@
 P 3650 5700
 F 0 "R3" H 3720 5746 50  0000 L CNN
-F 1 "R" H 3720 5655 50  0000 L CNN
+F 1 "5k1" H 3720 5655 50  0000 L CNN
 F 2 "Resistor_SMD:R_0402_1005Metric" V 3580 5700 50  0001 C CNN
 F 3 "~" H 3650 5700 50  0001 C CNN
@@
 P 4000 5700
 F 0 "R4" H 4070 5746 50  0000 L CNN
-F 1 "R" H 4070 5655 50  0000 L CNN
+F 1 "5k1" H 4070 5655 50  0000 L CNN
 F 2 "Resistor_SMD:R_0402_1005Metric" V 3930 5700 50  0001 C CNN
 F 3 "~" H 4000 5700 50  0001 C CNN
@@
 P 4050 1550
 F 0 "R8" V 3854 1550 50  0000 C CNN
-F 1 "DNP" V 3945 1550 50  0000 C CNN
+F 1 "0" V 3945 1550 50  0000 C CNN
 F 2 "Resistor_SMD:R_0402_1005Metric" H 4050 1550 50  0001 C CNN
 F 3 "~" H 4050 1550 50  0001 C CNN
@@
 P 4050 1650
 F 0 "R9" V 4154 1650 50  0000 C CNN
-F 1 "DNP" V 4245 1650 50  0000 C CNN
+F 1 "0" V 4245 1650 50  0000 C CNN
 F 2 "Resistor_SMD:R_0402_1005Metric" H 4050 1650 50  0001 C CNN
 F 3 "~" H 4050 1650 50  0001 C CNN
@@
 	1    0    0    -1
 $EndComp
-Text GLabel 3050 3300 0    50   Input ~ 0
+Text GLabel 2950 3300 0    50   Input ~ 0
 SDA
-Text GLabel 3050 3200 0    50   Input ~ 0
+Text GLabel 2950 3200 0    50   Input ~ 0
 SCL
-Text GLabel 3050 3400 0    50   Input ~ 0
+Text GLabel 2950 3400 0    50   Input ~ 0
 INT_N
 $Comp
@@
 	0    1    1    0
 $EndComp
+Wire Wire Line
+	2950 3200 3050 3200
+Wire Wire Line
+	3050 3300 2950 3300
+Wire Wire Line
+	2950 3400 3050 3400
+$Comp
+L power:+3V3 #PWR?
+U 1 1 5DA7B56B
+P 3300 4000
+F 0 "#PWR?" H 3300 3850 50  0001 C CNN
+F 1 "+3V3" H 3315 4173 50  0000 C CNN
+F 2 "" H 3300 4000 50  0001 C CNN
+F 3 "" H 3300 4000 50  0001 C CNN
+	1    3300 4000
+	1    0    0    -1
+$EndComp
 $EndSCHEMATC

Commit message: updated otterpill to V1.2
Parts:
- removed D3: SS310, Diode_SMD:D_SOD-123, symbol Device:D_Small
- removed U2: STM32F072CBUx, Package_DFN_QFN:QFN-48-1EP_7x7mm_P0.5mm_EP5.6x5.6mm, symbol MCU_ST_STM32F0:STM32F072CBUx
- removed U3: ACT4088, Package_TO_SOT_SMD:SOT-23-6, symbol otter:ACT4088
- added C11: 10u 25V, Capacitor_SMD:C_0805_2012Metric, symbol Device:C_Small
- added J2: VBUS, Connector_PinHeader_2.54mm:PinHeader_1x01_P2.54mm_Vertical, symbol Connector:Conn_01x01_Female
- added J6: GND, Connector_PinHeader_2.54mm:PinHeader_1x01_P2.54mm_Vertical, symbol Connector:Conn_01x01_Female
- added U2: STM32F072C8Tx, Package_QFP:LQFP-48_7x7mm_P0.5mm, symbol MCU_ST_STM32F0:STM32F072C8Tx
- added U3: SY8201, Package_TO_SOT_SMD:SOT-23-6, symbol otter:JW5026
- C1, C4: value 10u -> 10u 25V; LCSC (none) -> C15850
- C10, C2, C3, C5, C6, C7, C8, C9: value 100n -> 100n 50V
- D1: value LED -> LED RED
- D2: value LED -> LED GREEN
- R10, R11, R3, R4, R5, R7: value 5k1 -> 3k3
- R12: value 5k1 -> 10k
- R6: value 16k -> 10k
Connections:
- net +3V3: now also C11.1, U2.1 (VBAT), U2.24 (VDD), U2.36 (VDDIO2), U2.48 (VDD), U2.9 (VDDA); no longer R12.1
- net 31: now also U2.27 (PB14)
- net 310: now also U2.12 (PA2)
- net 311: now also U2.11 (PA1)
- net 312: now also U2.10 (PA0)
- net 313: now also U2.46 (PB9)
- net 314: now also U2.31 (PA10)
- net 315: now also U2.30 (PA9)
- net 32: now also U2.28 (PB15)
- net 33: now also U2.18 (PB0)
- net 35: now also U2.17 (PA7)
- net 36: now also U2.16 (PA6)
- net 37: now also U2.15 (PA5)
- net 38: now also U2.14 (PA4)
- net 39: now also U2.13 (PA3)
- net 41: now also U2.26 (PB13)
- net 410: now also U2.39 (PB3)
- net 411: now also U2.40 (PB4)
- net 413: now also U2.41 (PB5)
- net 43: now also U2.29 (PA8)
- net 44: now also U2.19 (PB1)
- net 45: now also U2.45 (PB8)
- net 46: now also U2.38 (PA15)
- net 47: now also U2.20 (PB2)
- net 48: now also U2.43 (PB7)
- net 49: now also U2.42 (PB6)
- net GND: now also C11.2, J6.1 (Pin_1), U2.23 (VSS), U2.35 (VSS), U2.47 (VSS), U2.8 (VSSA), U3.2 (GND)
- net INT_N: now also U2.25 (PB12); no longer R12.2
- net SCL: now also U2.21 (PB10)
- net SDA: now also U2.22 (PB11)
- net SWCLK: now also U2.37 (PA14)
- net SWDIO: now also U2.34 (PA13)
- net USB_N: now also U2.32 (PA11)
- net USB_P: now also U2.33 (PA12)
- net VBUS: now also J2.1 (Pin_1)
- net VIN: now also R12.1, U3.5 (VIN)
- net at R5.1, SW1.1: now also U2.2 (PC13), U2.44 (BOOT0)
- net at C3.2, L1.1: now also U3.6 (SW)
- net at R6.2, R7.1: now also U3.3 (FB)
- net at C3.1: now also U3.1 (BST)
- new net: R12.2, U3.4 (EN)
Other:
- moved on the sheet: C1, C2, C3, C4, C5, D4, L1, R10, R11, R6, R7

Commit message: updated otterpill to V1.2
Parts:
- L1: footprint Inductor_SMD:L_Taiyo-Yuden_MD-3030 -> Inductor_SMD:L_1210_3225Metric; LCSC (none) -> C86070
Changed lines of the file:
@@
 F 0 "L1" V 9385 1600 50  0000 C CNN
 F 1 "4u7" V 9294 1600 50  0000 C CNN
-F 2 "Inductor_SMD:L_Taiyo-Yuden_MD-3030" H 9200 1600 50  0001 C CNN
+F 2 "Inductor_SMD:L_1210_3225Metric" H 9200 1600 50  0001 C CNN
 F 3 "~" H 9200 1600 50  0001 C CNN
+F 4 "C86070" V 9200 1600 50  0001 C CNN "LCSC"
 	1    9200 1600
 	0    -1   -1   0
