File: HW v1.2/OtterPill.kicad_pcb (KiCad board)
At the start: 2 copper layers, 43.2 x 17.6 mm, 37 parts, among them J1 USB-c, J2 VBUS, J3 1, J4 2, J5 SWD, J6 GND, SW1 SW_Push, U1 USBLC6-4, U2 STM32F072C8Tx, U3 SY8201, U4 FUSB302BMPX

Commit message: updated V1.2
Parts:
- added G***: LOGO, otter:otter_laying_3411, B.Cu at (41.0, 26.8)
- added J7: PAD, TestPoint:TestPoint_Pad_1.0x1.0mm, B.Cu at (53.9, 33.3)
- added R13: 100, Resistor_SMD:R_0402_1005Metric, F.Cu at (49.8, 33.1)
- C2: footprint Capacitor_SMD:C_0402_1005Metric -> Capacitor_SMD:C_0603_1608Metric
- J5: footprint Connector_PinHeader_2.54mm:PinHeader_1x04_P2.54mm_Horizontal -> otter:PinHeader_1x04_P2.54mm_Horizontal
- moved R5 1.40 mm to (48.8, 33.1)
- moved C2 0.34 mm to (51.2, 29.3)
- moved R6 0.30 mm to (49.9, 29.0)
- moved C5 0.08 mm to (49.9, 31.0)
Connections:
- R5 pad 1: Net-(R5-Pad1) -> Net-(J7-Pad1)
- SW1 pad 1: Net-(R5-Pad1) -> Net-(R13-Pad1)
- U2 pad 2: Net-(R5-Pad1) -> Net-(J7-Pad1)
- U2 pad 44: Net-(R5-Pad1) -> Net-(J7-Pad1)
Routing:
- net Net-(R5-Pad1): track 16.9 -> 0.00 mm, vias 2 -> 0
- net Net-(J7-Pad1): track 0.00 -> 14.8 mm, vias 0 -> 3
- net Net-(R13-Pad1): track 0.00 -> 6.95 mm
- net GND: vias 41 -> 98
Other:
- rule pad_to_mask_clearance: 0.051 -> 0.01
- rule solder_mask_min_width: 0.25 -> 0.01
- board text added: "Jan Henrik 2019 v1.2"
- board text added: "Otter- Pill"
- board text removed: "Jan Henrik 2019"
