File: HW v1.2/OtterPill.kicad_pcb (KiCad board)
At the start: 2 copper layers, 43.2 x 17.6 mm, 40 parts, among them J1 USB-c, J2 VBUS, J3 1, J4 2, J5 SWD, J6 GND, J7 PAD, SW1 SW_Push, U1 USBLC6-4, U2 STM32F072C8Tx, U3 SY8201, U4 FUSB302BMPX

Commit message: schematic cleanup
Parts:
- R12, R6: value 10k -> 100k
- R7: value 3k3 -> 22k
- SW1: value SW_Push -> DFU
Connections:
- net 31 renamed PB14
- net 310 renamed PA2
- net 311 renamed PA1
- net 312 renamed PA0
- net 313 renamed PB9
- net 314 renamed PA10
- net 315 renamed PA9
- net 32 renamed PB15
- net 33 renamed PB0
- net 35 renamed PA7
- net 36 renamed PA6
- net 37 renamed PA5
- net 38 renamed PA4
- net 39 renamed PA3
- net 41 renamed PB13
- net 410 renamed PB3
- net 411 renamed PB4
- net 413 renamed PB5
- net 43 renamed PA8
- net 44 renamed PB1
- net 45 renamed PB8
- net 46 renamed PA15
- net 47 renamed PB2
- net 48 renamed PB7
- net 49 renamed PB6
