File: HW v1.2/OtterPill.sch (KiCad schematic (older format))
At the start: 37 parts, among them J1 USB-c, J2 VBUS, J3 1, J4 2, J5 SWD, J6 GND, SW1 SW_Push, U1 USBLC6-4, U2 STM32F072C8Tx, U3 SY8201, U4 FUSB302BMPX

Commit message: updated V1.2
Parts:
- added J7: PAD, TestPoint:TestPoint_Pad_1.0x1.0mm, symbol Connector:Conn_01x01_Female
- added R13: 100, Resistor_SMD:R_0402_1005Metric, symbol Device:R_Small
- C2: footprint Capacitor_SMD:C_0402_1005Metric -> Capacitor_SMD:C_0603_1608Metric
- J5: footprint Connector_PinHeader_2.54mm:PinHeader_1x04_P2.54mm_Horizontal -> otter:PinHeader_1x04_P2.54mm_Horizontal
Connections:
- net at R5.1, U2.2 (PC13), U2.44 (BOOT0): now also J7.1 (Pin_1), R13.2; no longer SW1.1
- new net: R13.1, SW1.1
Other:
- moved on the sheet: SW1
Changed lines of the file:
@@
 L Switch:SW_Push SW1
 U 1 1 5CC6C487
-P 4350 2500
-F 0 "SW1" V 4396 2452 50  0000 R CNN
-F 1 "SW_Push" V 4305 2452 50  0000 R CNN
-F 2 "Button_Switch_SMD:SW_SPST_PTS810" H 4350 2700 50  0001 C CNN
-F 3 "~" H 4350 2700 50  0001 C CNN
-	1    4350 2500
+P 4350 2300
+F 0 "SW1" V 4396 2252 50  0000 R CNN
+F 1 "SW_Push" V 4305 2252 50  0000 R CNN
+F 2 "Button_Switch_SMD:SW_SPST_PTS810" H 4350 2500 50  0001 C CNN
+F 3 "~" H 4350 2500 50  0001 C CNN
+	1    4350 2300
 	0    -1   -1   0
 $EndComp
@@
 L power:+3V3 #PWR0104
 U 1 1 5CC6C830
-P 4350 2300
-F 0 "#PWR0104" H 4350 2150 50  0001 C CNN
-F 1 "+3V3" H 4365 2473 50  0000 C CNN
-F 2 "" H 4350 2300 50  0001 C CNN
-F 3 "" H 4350 2300 50  0001 C CNN
-	1    4350 2300
+P 4350 2100
+F 0 "#PWR0104" H 4350 1950 50  0001 C CNN
+F 1 "+3V3" H 4365 2273 50  0000 C CNN
+F 2 "" H 4350 2100 50  0001 C CNN
+F 3 "" H 4350 2100 50  0001 C CNN
+	1    4350 2100
 	1    0    0    -1
 $EndComp
@@
 F 0 "C2" H 7642 1796 50  0000 L CNN
 F 1 "100n 50V" H 7642 1705 50  0000 L CNN
-F 2 "Capacitor_SMD:C_0402_1005Metric" H 7550 1750 50  0001 C CNN
+F 2 "Capacitor_SMD:C_0603_1608Metric" H 7550 1750 50  0001 C CNN
 F 3 "~" H 7550 1750 50  0001 C CNN
 	1    7550 1750
@@
 F 0 "J5" H 6758 5981 50  0000 C CNN
 F 1 "SWD" H 6758 5890 50  0000 C CNN
-F 2 "Connector_PinHeader_2.54mm:PinHeader_1x04_P2.54mm_Horizontal" H 6650 5700 50  0001 C CNN
+F 2 "otter:PinHeader_1x04_P2.54mm_Horizontal" H 6650 5700 50  0001 C CNN
 F 3 "~" H 6650 5700 50  0001 C CNN
 	1    6650 5700
@@
 Text GLabel 7350 1600 1    50   Input ~ 0
 VIN
+$Comp
+L Connector:Conn_01x01_Female J7
+U 1 1 5DB0ECB3
+P 4100 2700
+F 0 "J7" H 3994 2475 50  0000 C CNN
+F 1 "PAD" H 3994 2566 50  0000 C CNN
+F 2 "TestPoint:TestPoint_Pad_1.0x1.0mm" H 4100 2700 50  0001 C CNN
+F 3 "~" H 4100 2700 50  0001 C CNN
+	1    4100 2700
+	-1   0    0    1
+$EndComp
+Wire Wire Line
+	4300 2700 4350 2700
+$Comp
+L Device:R_Small R13
+U 1 1 5DB13626
+P 4350 2600
+F 0 "R13" H 4409 2646 50  0000 L CNN
+F 1 "100" H 4409 2555 50  0000 L CNN
+F 2 "Resistor_SMD:R_0402_1005Metric" H 4350 2600 50  0001 C CNN
+F 3 "~" H 4350 2600 50  0001 C CNN
+	1    4350 2600
+	1    0    0    -1
+$EndComp
 $EndSCHEMATC
