File: HW vG1.0/OtterPillG.kicad_pcb (KiCad board)
At the start: 2 copper layers, 43.2 x 17.6 mm, 35 parts, among them J1 USB-c, J2 VBUS, J3 1, J4 2, J5 SWD, J6 GND, SW1 DFU, U1 USBLC6-4, U2 STM32G071C8Tx, U3 SY8201, U4 CJ431

Commit message: updated vG1.0
Parts:
- added C8: 100n 50V, otter:C_0402, F.Cu at (49.0, 16.8)
- added R10: 100k, otter:R_0402, F.Cu at (51.4, 16.8)
- added R11: 3k3, otter:R_0402, F.Cu at (51.4, 18.4)
Changed lines of the file:
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@@
     (tracks 608)
     (zones 0)
-    (modules 35)
+    (modules 38)
     (nets 57)
   )
@@
     (uvia_dia 0.3)
     (uvia_drill 0.1)
+  )
+  (module otter:R_0402 (layer F.Cu)
+    (at 51.39 18.35)
+    (descr "Resistor 0402")
+    (tags "R Resistor 0805")
+    (attr smd)
+    (fp_text reference R11 (at 0 -0.75) (layer F.SilkS)
+      (effects (font (size 0.45 0.45) (thickness 0.1)))
+    )
+    (fp_text value 3k3 (at 0 -1.325) (layer F.Fab) hide
+      (effects (font (size 1 1) (thickness 0.15)))
+    )
+    (fp_line (start 0 0.15) (end 0 -0.15) (layer F.SilkS) (width 0.12))
+    (pad 2 smd rect (at 0.47 0) (size 0.5 0.6) (layers F.Cu F.Paste F.Mask)
+      (net 1 GND))
+    (pad 1 smd rect (at -0.47 0) (size 0.5 0.6) (layers F.Cu F.Paste F.Mask)
+      (net 44 PA0))
+    (model ${KISYS3DMOD}/Resistor_SMD.3dshapes/R_0402_1005Metric.step
+      (at (xyz 0 0 0))
+      (scale (xyz 1 1 1))
+      (rotate (xyz 0 0 0))
+    )
+  )
+  (module otter:R_0402 (layer F.Cu)
+    (at 51.39 16.75)
+    (descr "Resistor 0402")
+    (tags "R Resistor 0805")
+    (attr smd)
+    (fp_text reference R10 (at 0 -0.75) (layer F.SilkS)
+      (effects (font (size 0.45 0.45) (thickness 0.1)))
+    )
+    (fp_text value 100k (at 0 -1.325) (layer F.Fab) hide
+      (effects (font (size 1 1) (thickness 0.15)))
+    )
+    (fp_line (start 0 0.15) (end 0 -0.15) (layer F.SilkS) (width 0.12))
+    (pad 2 smd rect (at 0.47 0) (size 0.5 0.6) (layers F.Cu F.Paste F.Mask)
+      (net 44 PA0))
+    (pad 1 smd rect (at -0.47 0) (size 0.5 0.6) (layers F.Cu F.Paste F.Mask)
+      (net 17 VIN))
+    (model ${KISYS3DMOD}/Resistor_SMD.3dshapes/R_0402_1005Metric.step
+      (at (xyz 0 0 0))
+      (scale (xyz 1 1 1))
+      (rotate (xyz 0 0 0))
+    )
+  )
+  (module otter:C_0402 (layer F.Cu)
+    (at 48.95 16.75)
+    (descr "Capacitor 0402")
+    (tags "C Capacitor 0402")
+    (attr smd)
+    (fp_text reference C8 (at 0 -0.75) (layer F.SilkS)
+      (effects (font (size 0.45 0.45) (thickness 0.1)))
+    )
+    (fp_text value "100n 50V" (at 0 -1.325) (layer F.Fab) hide
+      (effects (font (size 1 1) (thickness 0.15)))
+    )
+    (fp_line (start 0 0.15) (end 0 -0.15) (layer F.SilkS) (width 0.12))
+    (pad 2 smd rect (at 0.47 0) (size 0.5 0.6) (layers F.Cu F.Paste F.Mask)
+      (net 1 GND))
+    (pad 1 smd rect (at -0.47 0) (size 0.5 0.6) (layers F.Cu F.Paste F.Mask)
+      (net 44 PA0))
+    (model ${KISYS3DMOD}/Capacitor_SMD.3dshapes/C_0402_1005Metric.step
+      (at (xyz 0 0 0))
+      (scale (xyz 1 1 1))
+      (rotate (xyz 0 0 0))
+    )
   )
   (module otter:R_0402 (layer F.Cu)
@@
   (segment (start 23.75 26.1) (end 24.46 26.81) (width 0.8) (layer F.Cu) (net 17))
   (via (at 24.77 29.6) (size 0.6) (drill 0.3) (layers F.Cu B.Cu) (net 17))
-  (segment (start 52.08 26.48) (end 52.96 26.48) (width 0.6) (layer F.Cu) (net 45))
-  (segment (start 51.972999 26.587001) (end 52.08 26.48) (width 0.6) (layer F.Cu) (net 45))
-  (segment (start 51.972999 27.894603) (end 51.972999 26.587001) (width 0.6) (layer F.Cu) (net 45))
-  (segment (start 51.8 28.235) (end 51.8 28.067602) (width 0.6) (layer F.Cu) (net 45))
-  (segment (start 52.315 28.75) (end 51.8 28.235) (width 0.6) (layer F.Cu) (net 45))
-  (segment (start 51.8 28.067602) (end 51.972999 27.894603) (width 0.6) (layer F.Cu) (net 45))
   (segment (start 59.26 35.527602) (end 59.26 36.1) (width 0.6) (layer B.Cu) (net 17))
-  (segment (start 51.972999 26.372999) (end 52.08 26.48) (width 0.6) (layer F.Cu) (net 45))
-  (segment (start 51.972999 24.965417) (end 51.972999 26.372999) (width 0.6) (layer F.Cu) (net 45))
-  (segment (start 52.4175 23.89) (end 52.4175 24.520916) (width 0.6) (layer F.Cu) (net 45))
-  (segment (start 52.4175 24.520916) (end 51.972999 24.965417) (width 0.6) (layer F.Cu) (net 45))
-  (segment (start 51.373058 28.494544) (end 51.500001 28.367601) (width 0.6) (layer F.Cu) (net 45))
-  (segment (start 51.500001 28.367601) (end 51.8 28.067602) (width 0.6) (layer F.Cu) (net 45))
   (via (at 24.3 30.45) (size 0.6) (drill 0.3) (layers F.Cu B.Cu) (net 17))
   (via (at 24.46 26.81) (size 0.6) (drill 0.3) (layers F.Cu B.Cu) (net 17))
@@
   (segment (start 23.65 26) (end 24.46 26.81) (width 0.8) (layer B.Cu) (net 17))
   (segment (start 23.65 24.01) (end 23.65 26) (width 0.8) (layer B.Cu) (net 17))
-  (segment (start 53.285 27.755) (end 52.96 27.43) (width 0.4) (layer F.Cu) (net 18))
-  (segment (start 53.285 28.75) (end 53.285 27.755) (width 0.4) (layer F.Cu) (net 18))
   (via (at 46.3 23.6) (size 0.6) (drill 0.3) (layers F.Cu B.Cu) (net 17))
   (segment (start 46.3 23.6) (end 46.3 24.3) (width 0.6) (layer B.Cu) (net 17))
@@
   (segment (start 53.700006 31.000006) (end 53.700006 34.76353) (width 0.4) (layer B.Cu) (net 17))
   (segment (start 59.26 36.1) (end 57.92353 34.76353) (width 0.4) (layer F.Cu) (net 17))
+  (segment (start 53.285 27.755) (end 52.96 27.43) (width 0.4) (layer F.Cu) (net 18))
+  (segment (start 53.285 28.75) (end 53.285 27.755) (width 0.4) (layer F.Cu) (net 18))
   (segment (start 56.773 33.585) (end 56.775 33.587) (width 0.157) (layer F.Cu) (net 19))
   (segment (start 50.140989 33.885989) (end 52.326011 33.885989) (width 0.157) (layer F.Cu) (net 19))
@@
   (segment (start 34.764653 31.201996) (end 33.678004 31.201996) (width 0.157) (layer F.Cu) (net 43))
   (segment (start 35.194618 30.772031) (end 34.764653 31.201996) (width 0.157) (layer F.Cu) (net 43))
+  (segment (start 52.08 26.48) (end 52.96 26.48) (width 0.6) (layer F.Cu) (net 45))
+  (segment (start 51.972999 26.587001) (end 52.08 26.48) (width 0.6) (layer F.Cu) (net 45))
+  (segment (start 51.972999 27.894603) (end 51.972999 26.587001) (width 0.6) (layer F.Cu) (net 45))
+  (segment (start 51.8 28.235) (end 51.8 28.067602) (width 0.6) (layer F.Cu) (net 45))
+  (segment (start 52.315 28.75) (end 51.8 28.235) (width 0.6) (layer F.Cu) (net 45))
+  (segment (start 51.8 28.067602) (end 51.972999 27.894603) (width 0.6) (layer F.Cu) (net 45))
+  (segment (start 51.972999 26.372999) (end 52.08 26.48) (width 0.6) (layer F.Cu) (net 45))
+  (segment (start 51.972999 24.965417) (end 51.972999 26.372999) (width 0.6) (layer F.Cu) (net 45))
+  (segment (start 52.4175 23.89) (end 52.4175 24.520916) (width 0.6) (layer F.Cu) (net 45))
+  (segment (start 52.4175 24.520916) (end 51.972999 24.965417) (width 0.6) (layer F.Cu) (net 45))
+  (segment (start 51.373058 28.494544) (end 51.500001 28.367601) (width 0.6) (layer F.Cu) (net 45))
+  (segment (start 51.500001 28.367601) (end 51.8 28.067602) (width 0.6) (layer F.Cu) (net 45))
   (segment (start 51.34 22.7) (end 52.53 23.89) (width 0.6) (layer F.Cu) (net 45))
   (segment (start 50 22.7) (end 51.34 22.7) (width 0.6) (layer F.Cu) (net 45))
