File: HW vG1.0/OtterPillG.sch (KiCad schematic (older format))
At the start: 36 parts, among them J1 USB-c, J2 VBUS, J3 1, J4 2, J5 SWD, J6 GND, SW1 DFU, U1 USBLC6-4, U2 STM32G071C8Tx, U3 SY8201, U4 CJ431

Commit message: updated vG1.0
Parts:
- removed C10: 100n 50V, otter:C_0402, symbol Device:C_Small
- added R10: 100k, otter:R_0402, symbol Device:R_Small
- added R11: 3k3, otter:R_0402, symbol Device:R
Connections:
- net +3V3: no longer C8.1
- net GND: now also R11.2
- net PA0: now also C8.1, R10.2, R11.1
- net VBUS: now also R10.1
Other:
- moved on the sheet: C8
Changed lines of the file:
@@
-	1    0    0    -1
-$EndComp
-$Comp
-L Device:C_Small C10
-U 1 1 5CC9C524
-P 3200 7150
-F 0 "C10" H 3292 7196 50  0000 L CNN
-F 1 "100n 50V" H 3292 7105 50  0000 L CNN
-F 2 "otter:C_0402" H 3200 7150 50  0001 C CNN
-F 3 "~" H 3200 7150 50  0001 C CNN
-	1    3200 7150
-	1    0    0    -1
-$EndComp
-$Comp
-L power:GND #PWR0143
-U 1 1 5CC9C530
-P 3200 7250
-F 0 "#PWR0143" H 3200 7000 50  0001 C CNN
-F 1 "GND" H 3205 7077 50  0000 C CNN
-F 2 "" H 3200 7250 50  0001 C CNN
-F 3 "" H 3200 7250 50  0001 C CNN
-	1    3200 7250
-	1    0    0    -1
-$EndComp
-$Comp
-L power:VBUS #PWR0144
-U 1 1 5CC9D5C7
-P 3200 7050
-F 0 "#PWR0144" H 3200 6900 50  0001 C CNN
-F 1 "VBUS" H 3215 7223 50  0000 C CNN
-F 2 "" H 3200 7050 50  0001 C CNN
-F 3 "" H 3200 7050 50  0001 C CNN
-	1    3200 7050
 	1    0    0    -1
 $EndComp
@@
 L power:GND #PWR0140
 U 1 1 5CC9B0F8
-P 2100 7250
-F 0 "#PWR0140" H 2100 7000 50  0001 C CNN
-F 1 "GND" H 2105 7077 50  0000 C CNN
-F 2 "" H 2100 7250 50  0001 C CNN
-F 3 "" H 2100 7250 50  0001 C CNN
-	1    2100 7250
-	1    0    0    -1
-$EndComp
-$Comp
-L power:+3V3 #PWR0139
-U 1 1 5CC9B0F2
-P 2100 7050
-F 0 "#PWR0139" H 2100 6900 50  0001 C CNN
-F 1 "+3V3" H 2115 7223 50  0000 C CNN
-F 2 "" H 2100 7050 50  0001 C CNN
-F 3 "" H 2100 7050 50  0001 C CNN
-	1    2100 7050
+P 4150 4000
+F 0 "#PWR0140" H 4150 3750 50  0001 C CNN
+F 1 "GND" H 4155 3827 50  0000 C CNN
+F 2 "" H 4150 4000 50  0001 C CNN
+F 3 "" H 4150 4000 50  0001 C CNN
+	1    4150 4000
 	1    0    0    -1
 $EndComp
@@
 L Device:C_Small C8
 U 1 1 5CC9B0EC
-P 2100 7150
-F 0 "C8" H 2192 7196 50  0000 L CNN
-F 1 "100n 50V" H 2192 7105 50  0000 L CNN
-F 2 "otter:C_0402" H 2100 7150 50  0001 C CNN
-F 3 "~" H 2100 7150 50  0001 C CNN
-	1    2100 7150
-	1    0    0    -1
-$EndComp
+P 4150 3900
+F 0 "C8" H 4242 3946 50  0000 L CNN
+F 1 "100n 50V" H 4242 3855 50  0000 L CNN
+F 2 "otter:C_0402" H 4150 3900 50  0001 C CNN
+F 3 "~" H 4150 3900 50  0001 C CNN
+	1    4150 3900
+	1    0    0    -1
+$EndComp
+$Comp
+L Device:R_Small R10
+U 1 1 5F9ACC9B
+P 3800 3550
+F 0 "R10" H 3859 3596 50  0000 L CNN
+F 1 "100k" H 3859 3505 50  0000 L CNN
+F 2 "otter:R_0402" H 3800 3550 50  0001 C CNN
+F 3 "~" H 3800 3550 50  0001 C CNN
+	1    3800 3550
+	1    0    0    -1
+$EndComp
+$Comp
+L Device:R R11
+U 1 1 5F9ADF8B
+P 3800 3900
+F 0 "R11" H 3870 3946 50  0000 L CNN
+F 1 "3k3" H 3870 3855 50  0000 L CNN
+F 2 "otter:R_0402" V 3730 3900 50  0001 C CNN
+F 3 "~" H 3800 3900 50  0001 C CNN
+	1    3800 3900
+	1    0    0    -1
+$EndComp
+Text GLabel 4200 3700 2    50   Input ~ 0
+PA0
+$Comp
+L power:VBUS #PWR0135
+U 1 1 5F9B01BD
+P 3800 3450
+F 0 "#PWR0135" H 3800 3300 50  0001 C CNN
+F 1 "VBUS" H 3815 3623 50  0000 C CNN
+F 2 "" H 3800 3450 50  0001 C CNN
+F 3 "" H 3800 3450 50  0001 C CNN
+	1    3800 3450
+	1    0    0    -1
+$EndComp
+$Comp
+L power:GND #PWR0136
+U 1 1 5F9B1249
+P 3800 4050
+F 0 "#PWR0136" H 3800 3800 50  0001 C CNN
+F 1 "GND" H 3805 3877 50  0000 C CNN
+F 2 "" H 3800 4050 50  0001 C CNN
+F 3 "" H 3800 4050 50  0001 C CNN
+	1    3800 4050
+	1    0    0    -1
+$EndComp
+Wire Wire Line
+	3800 3700 3800 3750
+Wire Wire Line
+	3800 3700 3800 3650
+Connection ~ 3800 3700
+Wire Wire Line
+	3800 3700 4150 3700
+Wire Wire Line
+	4150 3800 4150 3700
+Connection ~ 4150 3700
+Wire Wire Line
+	4150 3700 4200 3700
 $EndSCHEMATC
